File: keyboard/hardware/keyboard-controller/analog_input.kicad_sch (KiCad schematic)
At the start: 41 parts, among them SW11 CLK_DIV, SW12 SUB_MODE, U10 CD4051B

Commit message: Partially converted keyboard libaries over to common dir
Parts:
- RV1, RV2, RV3: footprint Alpha_Potentiometers:Potentiometer_Alpha_RV09AF-40-20K-B1K_Single_Vertical -> Alpha_Pots:Potentiometer_Alpha_RV09AF-40-20K_Single_Vertical
Changed lines of the file:
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@@
       (effects (font (size 1.27 1.27)) (justify right))
     )
-    (property "Footprint" "Alpha_Potentiometers:Potentiometer_Alpha_RV09AF-40-20K-B1K_Single_Vertical" (id 2) (at 151.13 80.01 0)
+    (property "Footprint" "Alpha_Pots:Potentiometer_Alpha_RV09AF-40-20K_Single_Vertical" (id 2) (at 151.13 80.01 0)
       (effects (font (size 1.27 1.27)) hide)
     )
@@
       (effects (font (size 1.27 1.27)) (justify right))
     )
-    (property "Footprint" "Alpha_Potentiometers:Potentiometer_Alpha_RV09AF-40-20K-B1K_Single_Vertical" (id 2) (at 151.13 36.83 0)
+    (property "Footprint" "Alpha_Pots:Potentiometer_Alpha_RV09AF-40-20K_Single_Vertical" (id 2) (at 151.13 36.83 0)
       (effects (font (size 1.27 1.27)) hide)
     )
@@
       (effects (font (size 1.27 1.27)) (justify right))
     )
-    (property "Footprint" "Alpha_Potentiometers:Potentiometer_Alpha_RV09AF-40-20K-B1K_Single_Vertical" (id 2) (at 151.13 127 0)
+    (property "Footprint" "Alpha_Pots:Potentiometer_Alpha_RV09AF-40-20K_Single_Vertical" (id 2) (at 151.13 127 0)
       (effects (font (size 1.27 1.27)) hide)
     )
