File: keyboard/hardware/keyboard-controller/keyboard-controller.kicad_pcb (KiCad board)
At the start: 2 copper layers, 257 x 195 mm, 119 parts, among them J1 Debug_Pins, J2 Barrel_Jack_Switch, J3 Keybed Connector, J4 SYNC_IN, J5 CV_OUT, J6 GATE_OUT, J7 SYNC_OUT, Q1 2N3904, SW1 RESET, SW10 FUNCTION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

Commit message: Partially converted keyboard libaries over to common dir
Parts:
- R11: value 1k -> 1K
- RV1, RV2, RV3: footprint Alpha_Potentiometers:Potentiometer_Alpha_RV09AF-40-20K-B1K_Single_Vertical -> Alpha_Pots:Potentiometer_Alpha_RV09AF-40-20K_Single_Vertical
- SW10: value FUNCTION -> REST
- SW6: value RECORD -> STOP
- SW7: value STOP -> RECORD
- SW8: value REST -> HOLD
- SW9: value HOLD -> FUNC
- U4: value TL431LP -> TL431
- turned RV1 to 0 degrees
- turned RV2 to 0 degrees
- turned RV3 to 0 degrees

Commit message: Simplified keyboard for rev1
Parts:
- removed C11, C12, C13, C14, C15, C16, C17, C18, C19, C20, C21: 0.1uF, AEC_Capacitors:C_Disc_D5.0mm_W2.5mm_P3.0mm
- removed D15, D16: 1N5818, Diode_THT:D_DO-41_SOD81_P10.16mm_Horizontal
- removed J4: SYNC_IN, AudioJacks:Jack_3.5mm_QingPu_WQP-PJ398SM_Vertical
- removed J7: SYNC_OUT, AudioJacks:Jack_3.5mm_QingPu_WQP-PJ398SM_Vertical
- removed Q1: 2N3904, Package_TO_SOT_THT:TO-92_Inline
- removed R10, R9: 1M, Royal_Ohm_Resistors:R_Axial_DIN0207_L6.8mm_D2.5mm_P10.16mm_Horizontal
- removed R11, R20, R7: 1K, Royal_Ohm_Resistors:R_Axial_DIN0207_L6.8mm_D2.5mm_P10.16mm_Horizontal
- removed R14: 20K, Royal_Ohm_Resistors:R_Axial_DIN0207_L6.8mm_D2.5mm_P10.16mm_Horizontal
- removed R17: 10K, Royal_Ohm_Resistors:R_Axial_DIN0207_L6.8mm_D2.5mm_P10.16mm_Horizontal
- removed R21, R22, R23, R24, R25, R26, R27, R28, R29, R30, R31, R32, R33, R34, R35, R36, R37, R38, R39, R40, R41, R42, R43, R44: 2.2K, Royal_Ohm_Resistors:R_Axial_DIN0207_L6.8mm_D2.5mm_P10.16mm_Horizontal
- removed R8: 100K, Royal_Ohm_Resistors:R_Axial_DIN0207_L6.8mm_D2.5mm_P10.16mm_Horizontal
- removed REF**: Polarity_Center_Positive_6mm_SilkScreen, Symbol:Polarity_Center_Positive_6mm_SilkScreen
- removed RV1: CLK_SPEED, Alpha_Pots:Potentiometer_Alpha_RV09AF-40-20K_Single_Vertical
- removed RV2: PORTAMENTO, Alpha_Pots:Potentiometer_Alpha_RV09AF-40-20K_Single_Vertical
- removed RV3: GATE_TIME, Alpha_Pots:Potentiometer_Alpha_RV09AF-40-20K_Single_Vertical
- removed SW11: CLK_DIV, Keyboard:Clock_Div_Switch
- removed SW12: SUB_MODE, Keyboard:Sub_Mode_Switch
- removed SW2: MODE_SEL, Wealth_Metal_Switches:Slide_Switch_SPDT_SS12F44G5
- removed U10: CD4051B, Package_DIP:DIP-16_W7.62mm_Socket
- moved H3 324.1 mm to (75.6, 239.5)
- moved J2 293.0 mm to (51.2, 112.8), turned to 0 degrees
- moved H2 267.1 mm to (76.6, 260.1)
- moved C6 261.2 mm to (71.3, 102.9), turned to 0 degrees
- moved U5 261.1 mm to (67.1, 102.2)
- moved C5 260.3 mm to (71.3, 97.1)
- moved C3 233.0 mm to (58.6, 117.3)
- moved J1 231.4 mm to (117.4, 118.4), turned to 180 degrees
- moved D6 231.3 mm to (59.6, 123.9), turned to 0 degrees
- moved U3 217.8 mm to (66.4, 110.4), turned to 180 degrees
- moved R2 213.0 mm to (258.3, 61.7), turned to 0 degrees
- moved C4 205.2 mm to (71.4, 116.2), turned to 180 degrees
- moved D3 200.9 mm to (282.6, 79.3)
- moved D2 195.8 mm to (251.2, 71.7)
- moved H4 191.3 mm to (62.2, 241.4)
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Connections:
- R16 pad 2: Net-(R16-Pad2) -> Net-(U8-Pad5)
- R18 pad 1: Net-(R16-Pad2) -> Net-(R18-Pad1)
- R19 pad 1: Net-(R15-Pad2) -> Net-(U8-Pad2)
- U1 pad 10: /AN_ADDR_B -> unconnected-(U1-Pad10)
- U1 pad 11: /AN_ADDR_C -> unconnected-(U1-Pad11)
- U1 pad 29: /MODE_SEL -> unconnected-(U1-Pad29)
- U1 pad 31: /ANALOG_IN -> unconnected-(U1-Pad31)
- U1 pad 4: /SYNC_CN -> unconnected-(U1-Pad4)
- U1 pad 5: /SYNC_IN -> unconnected-(U1-Pad5)
- U1 pad 6: /SYNC_OUT -> unconnected-(U1-Pad6)
- U1 pad 9: /AN_ADDR_A -> unconnected-(U1-Pad9)
- U8 pad 1: Net-(R17-Pad2) -> Net-(U8-Pad2)
- U8 pad 2: Net-(R14-Pad1) -> Net-(U8-Pad2)
- U8 pad 3: /SYNC_OUT -> Net-(R15-Pad2)
- U8 pad 5: GND -> Net-(U8-Pad5)
- U8 pad 6: Net-(U8-Pad6) -> Net-(R18-Pad1)
- U8 pad 7: Net-(U8-Pad6) -> Net-(R18-Pad1)
- U9 pad 1: Net-(R16-Pad2) -> Net-(U8-Pad5)
Routing:
- net +3.3V: track 686.3 -> 0.00 mm, vias 1 -> 0
- net /Key Matrix/MATRIX_C1: track 199.5 -> 0.00 mm
- net /SWDIO: track 142.1 -> 0.00 mm
- net /SWDCLK: track 140.5 -> 0.00 mm
- net /LED1: track 137.0 -> 0.00 mm
- net /MATRIX_DATA: track 136.8 -> 0.00 mm
- net /MATRIX_R6: track 133.4 -> 0.00 mm
- net /MATRIX_R5: track 130.1 -> 0.00 mm
- net /MATRIX_R4: track 121.2 -> 0.00 mm
- net /LED2: track 119.0 -> 0.00 mm
- net /LED3: track 116.0 -> 0.00 mm
- net /MATRIX_CLK: track 111.3 -> 0.00 mm
- net /LED4: track 109.7 -> 0.00 mm
- net /MATRIX_R3: track 101.9 -> 0.00 mm
- net /Key Matrix/MATRIX_C10: track 101.1 -> 0.00 mm
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- removed copper zone on B.Cu, net GND
- removed copper zone on F.Cu, net GND
Other:
- board outline removed
- board text removed: "+"
- board text removed: "-"
- board text removed: "12V, 200mA"
- board text removed: "Arp"
- board text removed: "CV Out"
- board text removed: "Clock Division"
- board text removed: "Clock Speed"
- board text removed: "Func"
- board text removed: "GND"
- board text removed: "Gate Out"
- board text removed: "Gate Time"
- board text removed: "Hold"
- board text removed: "July, 2022"
- board text removed: "Keyboard Controller - REV1"
- board text removed: "Mode"
- board text removed: "Northridge Devices"
- board text removed: "Play/Pause"
- board text removed: "Portamento"
- board text removed: "Record"
- board text removed: "Reset"
- board text removed: "Rest"
- board text removed: "SERCLK"
- board text removed: "SERDATA"
- board text removed: "SWDCLK"
- board text removed: "SWDIO"
- board text removed: "Seq"
- board text removed: "Stop"
- board text removed: "Sync In"
- board text removed: "Sync Out"

Commit message: Finalized keyboard controller rev1 board
Parts:
- removed D10, D11, D12, D13, D14: 1N4148, Diode_THT:D_DO-35_SOD27_P7.62mm_Horizontal
- removed D5: LED4, LED_THT:LED_D5.0mm
- removed R5: 470, Royal_Ohm_Resistors:R_Axial_DIN0207_L6.8mm_D2.5mm_P10.16mm_Horizontal
- removed SW1: RESET, Button_Switch_THT:SW_PUSH_6mm
- removed SW10: REST, Button_Switch_THT:SW_PUSH_6mm
- removed SW6: STOP, Button_Switch_THT:SW_PUSH_6mm
- removed SW7: RECORD, Button_Switch_THT:SW_PUSH_6mm
- removed SW8: HOLD, Button_Switch_THT:SW_PUSH_6mm
- removed SW9: FUNC, Button_Switch_THT:SW_PUSH_6mm
- D2: value LED1 -> OCTAVE_DOWN_LED
- D3: value LED2 -> MIDDLE_OCTAVE_LED
- D4: value LED3 -> OCTAVE_UP_LED
- SW5: value PLAY_PAUSE -> FUNC
- moved H3 243.9 mm to (294.0, 131.0), turned to 90 degrees
- moved H4 238.8 mm to (294.0, 184.0), turned to 90 degrees
- moved C3 202.8 mm to (260.9, 131.4), turned to 90 degrees
- moved U3 196.4 mm to (260.9, 137.4), turned to 90 degrees
- moved D6 194.4 mm to (253.9, 131.3), turned to -90 degrees
- moved C4 192.4 mm to (262.1, 141.9)
- moved H1 136.7 mm to (111.0, 131.0), turned to 90 degrees
- moved R1 130.0 mm to (154.5, 142.1), turned to 90 degrees
- moved D3 123.1 mm to (174.5, 138.3), turned to 90 degrees
- moved D1 122.5 mm to (147.8, 138.3), turned to 90 degrees
- moved R2 121.0 mm to (167.8, 142.1), turned to 90 degrees
- moved J6 116.7 mm to (270.8, 148.0)
- moved D2 111.9 mm to (161.2, 138.3), turned to 90 degrees
- moved U8 111.2 mm to (251.8, 164.2)
- moved J3 107.5 mm to (196.0, 183.0), turned to 90 degrees
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Connections:
- J3 pad 16: unconnected-(J3-Pad16) -> GND
- R16 pad 2: Net-(U8-Pad5) -> Net-(R16-Pad2)
- U1 pad 16: /LED4 -> unconnected-(U1-Pad16)
- U1 pad 21: /MATRIX_R1 -> /MATRIX_DATA
- U1 pad 22: /MATRIX_R2 -> /MATRIX_CLK
- U1 pad 24: /MATRIX_R3 -> /MATRIX_R6
- U1 pad 25: /MATRIX_R4 -> /MATRIX_R5
- U1 pad 26: /MATRIX_R5 -> /MATRIX_R4
- U1 pad 27: /MATRIX_R6 -> /MATRIX_R3
- U1 pad 29: unconnected-(U1-Pad29) -> /MATRIX_R2
- U1 pad 30: /RUN -> unconnected-(U1-Pad30)
- U1 pad 31: unconnected-(U1-Pad31) -> /MATRIX_R1
- U1 pad 32: /MATRIX_CLK -> unconnected-(U1-Pad32)
- U1 pad 34: /MATRIX_DATA -> unconnected-(U1-Pad34)
- U7 pad 4: /Key Matrix/MATRIX_C10 -> unconnected-(U7-Pad4)
- U8 pad 5: Net-(U8-Pad5) -> /GATE_OUT
- U8 pad 6: Net-(R18-Pad1) -> Net-(R13-Pad1)
- U8 pad 7: Net-(R18-Pad1) -> Net-(R15-Pad2)
- U9 pad 1: Net-(U8-Pad5) -> Net-(R16-Pad2)
- U9 pad 5: /GATE_OUT -> Net-(R16-Pad2)
- U9 pad 6: Net-(R13-Pad1) -> Net-(R18-Pad1)
- U9 pad 7: Net-(R15-Pad2) -> Net-(R18-Pad1)
Routing:
- net +12V: track 0.00 -> 160.7 mm
- net /Key Matrix/MATRIX_C1: track 0.00 -> 84.8 mm
- net /MATRIX_R3: track 0.00 -> 70.5 mm
- net /Key Matrix/MATRIX_C9: track 0.00 -> 67.3 mm
- net /Key Matrix/MATRIX_C8: track 0.00 -> 57.9 mm
- net /MATRIX_R2: track 0.00 -> 57.8 mm
- net /MATRIX_R1: track 0.00 -> 51.5 mm
- net /GATE_OUT: track 0.00 -> 51.2 mm
- net /SWDIO: track 0.00 -> 46.8 mm
- net /SPI_DATA: track 0.00 -> 44.6 mm
- net /Key Matrix/MATRIX_C4: track 0.00 -> 43.9 mm
- net /MATRIX_CLK: track 0.00 -> 43.2 mm, vias 0 -> 1
- net /SPI_CLK: track 0.00 -> 41.8 mm
- net /CV_OUT: track 0.00 -> 37.8 mm
- net /DAC_CS: track 0.00 -> 37.0 mm
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- added copper zone on B.Cu, net +3.3V
- added copper zone on B.Cu, net +9V
- added copper zone on F.Cu, net GND
Other:
- board outline added: 195 x 65 mm
- board text added: "+O"
- board text added: "-O"
- board text added: "CV"
- board text added: "FUNC"
- board text added: "GATE"
- board text added: "GND"
- board text added: "Keyboard Controller - rev1"
- board text added: "Northridge Synth - 12/23"
- board text added: "O"
- board text added: "O+"
- board text added: "PWR"
- board text added: "SERDATA"
- board text added: "SWDCLK"
- board text added: "SWDIO"
