File: power-supply/power-supply.kicad_sch (KiCad schematic)
At the start: 25 parts, among them J1 Barrel_Jack_Switch, J2 Output, U1 LM7812_TO220, U2 LM7912_TO220

Commit message: Fixed capacitor polarity on power supply
Parts:
- C10, C7, C8, C9: symbol Device:C -> Device:C_Polarized_US
Connections:
- net GND: now also C10.1, C8.1; no longer C10.2, C8.2
- net at C2.2, C4.2, C6.2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: now also C8.2; no longer C8.1
- net at J2.1 (Pin_1), U2.3 (VO): now also C10.2; no longer C10.1
Changed lines of the file:
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@@
   (title_block
     (title "Eurorack Power Supply")
-    (rev "rev2")
+    (rev "rev3")
     (company "Northride Synth")
   )
@@
     (pin "2")
   )
-  (symbol (lib_id "Device:C") (at 162.56 110.49 0) (unit 1)
-    (in_bom yes) (on_board yes) (fields_autoplaced)
-    (property "Reference" "C8" (id 0) (at 166.37 109.2199 0)
-      (effects (font (size 1.27 1.27)) (justify left))
-    )
-    (property "Value" "2.2uF" (id 1) (at 166.37 111.7599 0)
-      (effects (font (size 1.27 1.27)) (justify left))
-    )
-    (property "Footprint" "Capacitor_THT:CP_Radial_Tantal_D5.0mm_P2.50mm" (id 2) (at 163.5252 114.3 0)
+  (symbol (lib_id "Device:C_Polarized_US") (at 162.56 110.49 0) (mirror x) (unit 1)
+    (in_bom yes) (on_board yes)
+    (property "Reference" "C8" (id 0) (at 168.91 109.22 0)
+      (effects (font (size 1.27 1.27)) (justify right))
+    )
+    (property "Value" "2.2uF" (id 1) (at 171.45 111.76 0)
+      (effects (font (size 1.27 1.27)) (justify right))
+    )
+    (property "Footprint" "Capacitor_THT:CP_Radial_Tantal_D5.0mm_P2.50mm" (id 2) (at 162.56 110.49 0)
       (effects (font (size 1.27 1.27)) hide)
     )
@@
     )
   )
-  (symbol (lib_id "Device:C") (at 162.56 80.01 0) (unit 1)
+  (symbol (lib_id "Device:C_Polarized_US") (at 162.56 80.01 0) (unit 1)
     (in_bom yes) (on_board yes) (fields_autoplaced)
     (property "Reference" "C7" (id 0) (at 166.37 78.7399 0)
@@
       (effects (font (size 1.27 1.27)) (justify left))
     )
-    (property "Footprint" "Capacitor_THT:CP_Radial_Tantal_D5.0mm_P2.50mm" (id 2) (at 163.5252 83.82 0)
+    (property "Footprint" "Capacitor_THT:CP_Radial_Tantal_D5.0mm_P2.50mm" (id 2) (at 162.56 80.01 0)
       (effects (font (size 1.27 1.27)) hide)
     )
@@
     (pin "3")
   )
-  (symbol (lib_id "Device:C") (at 196.85 110.49 0) (unit 1)
-    (in_bom yes) (on_board yes) (fields_autoplaced)
-    (property "Reference" "C10" (id 0) (at 200.66 109.2199 0)
-      (effects (font (size 1.27 1.27)) (justify left))
-    )
-    (property "Value" "1uF" (id 1) (at 200.66 111.7599 0)
-      (effects (font (size 1.27 1.27)) (justify left))
-    )
-    (property "Footprint" "Capacitor_THT:CP_Radial_Tantal_D5.0mm_P2.50mm" (id 2) (at 197.8152 114.3 0)
+  (symbol (lib_id "Device:C_Polarized_US") (at 196.85 110.49 0) (mirror x) (unit 1)
+    (in_bom yes) (on_board yes)
+    (property "Reference" "C10" (id 0) (at 204.47 109.22 0)
+      (effects (font (size 1.27 1.27)) (justify right))
+    )
+    (property "Value" "1uF" (id 1) (at 204.47 111.76 0)
+      (effects (font (size 1.27 1.27)) (justify right))
+    )
+    (property "Footprint" "Capacitor_THT:CP_Radial_Tantal_D5.0mm_P2.50mm" (id 2) (at 196.85 110.49 0)
       (effects (font (size 1.27 1.27)) hide)
     )
@@
     )
   )
-  (symbol (lib_id "Device:C") (at 196.85 80.01 0) (unit 1)
+  (symbol (lib_id "Device:C_Polarized_US") (at 196.85 80.01 0) (unit 1)
     (in_bom yes) (on_board yes) (fields_autoplaced)
     (property "Reference" "C9" (id 0) (at 200.66 78.7399 0)
@@
       (effects (font (size 1.27 1.27)) (justify left))
     )
-    (property "Footprint" "Capacitor_THT:CP_Radial_Tantal_D5.0mm_P2.50mm" (id 2) (at 197.8152 83.82 0)
-      (effects (font (size 1.27 1.27)) hide)
-    )
+    (property "Footprint" "Capacitor_THT:CP_Radial_Tantal_D5.0mm_P2.50mm" (id 2) (at 196.85 80.01 0)
+      (effects (font (size 1.27 1.27)) hide)
+    )
