File: sample-and-hold/sample-and-hold-panel/sample-and-hold-panel.kicad_pcb (KiCad board)
At the start: 2 copper layers, 20 x 128.5 mm, 6 parts

Commit message: Added revision text to sample and hold board/panel
Other:
- board text added: "Northridge Device - Sept 2022"
- board text added: "S&H - REV1"
- board text removed: "REV1"
Changed lines of the file:
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@@
   (gr_line (start 140 44.25) (end 160 44.25) (layer "Dwgs.User") (width 0.15))
   (gr_circle (center 150 52) (end 151.55 52) (layer "Edge.Cuts") (width 0.2) (fill none))
-  (gr_text "REV1" (at 157 157) (layer "B.SilkS")
+  (gr_text "Northridge Device - Sept 2022" (at 141.25 145.25 90) (layer "B.SilkS")
     (effects (font (size 1 1) (thickness 0.15)) (justify mirror))
   )
+  (gr_text "S&H - REV1" (at 158.5 152.75 90) (layer "B.SilkS")
+    (effects (font (size 1 1) (thickness 0.15)) (justify mirror))
+  )
