File: noise/noise/noise.kicad_sch (KiCad schematic)
At the start: 38 parts, among them J1 Power Connector, J2 WHITE_OUT, J3 BLUE_OUT, J4 PINK_OUT, Q1 BC548, U1 TL074

Commit message: Added footprints for noise module parts and created BOM
Parts:
- C11, C4: footprint (none) -> Capacitor_THT:C_Rect_L7.2mm_W2.5mm_P5.00mm_FKS2_FKP2_MKS2_MKP2; Manufacturer (none) -> ARCOTRONICS; Manufacturer Part No. (none) -> 5.6nF/100V; Supplier (none) -> Tayda; Supplier Part No. (none) -> A-423
- C3: footprint (none) -> Capacitor_THT:C_Rect_L7.2mm_W3.5mm_P5.00mm_FKS2_FKP2_MKS2_MKP2; Manufacturer (none) -> WIMA; Manufacturer Part No. (none) -> MKS2B041001C00KSSD; Supplier (none) -> Tayda; Supplier Part No. (none) -> A-3290
- C5, C8: footprint (none) -> Capacitor_THT:C_Rect_L7.2mm_W2.5mm_P5.00mm_FKS2_FKP2_MKS2_MKP2; Manufacturer (none) -> WIMA; Manufacturer Part No. (none) -> FKS2D012201A00JSSD; Supplier (none) -> Tayda; Supplier Part No. (none) -> A-935
- C6, C7: footprint (none) -> Capacitor_THT:C_Rect_L7.2mm_W5.5mm_P5.00mm_FKS2_FKP2_MKS2_MKP2; Manufacturer (none) -> WIMA; Manufacturer Part No. (none) -> FKP2O106801G00JSSD; Supplier (none) -> Mouser; Supplier Part No. (none) -> 505-FKP2680/1000/5
- J2, J3, J4: Manufacturer (none) -> Tayda; Manufacturer Part No. (none) -> PJ-323M; Supplier (none) -> Tayda; Supplier Part No. (none) -> A-2557
- Q1: Manufacturer (none) -> KEC; Manufacturer Part No. (none) -> BC548B; Supplier (none) -> Tayda; Supplier Part No. (none) -> A-141
- R10: footprint (none) -> Resistor_THT:R_Axial_DIN0207_L6.3mm_D2.5mm_P10.16mm_Horizontal; Manufacturer (none) -> Royal Ohm; Manufacturer Part No. (none) -> MF0W4FF4702A50; Supplier (none) -> Tayda; Supplier Part No. (none) -> A-2279
- R11: Manufacturer Part No. MF0W4FF1003A50 -> MF0W4FF2002A50; Supplier Part No. A-2248 -> A-2339
- R12: footprint (none) -> Resistor_THT:R_Axial_DIN0207_L6.3mm_D2.5mm_P10.16mm_Horizontal; Manufacturer (none) -> Royal Ohm; Manufacturer Part No. (none) -> MF0W4FF4703A50; Supplier (none) -> Tayda; Supplier Part No. (none) -> A-2180
- R13: footprint (none) -> Resistor_THT:R_Axial_DIN0207_L6.3mm_D2.5mm_P10.16mm_Horizontal; Manufacturer (none) -> Royal Ohm; Manufacturer Part No. (none) -> MF0W4FF1003A50; Supplier (none) -> Tayda; Supplier Part No. (none) -> A-2248
- R14: footprint (none) -> Resistor_THT:R_Axial_DIN0207_L6.3mm_D2.5mm_P10.16mm_Horizontal; Manufacturer (none) -> Royal Ohm; Manufacturer Part No. (none) -> MF0W4FF2202A50; Supplier (none) -> Tayda; Supplier Part No. (none) -> A-2339
- R15: Manufacturer Part No. MF0W4FF1003A50 -> MF0W4FF3302A50; Supplier Part No. A-2248 -> A-2290
- R17, R18, R19: footprint (none) -> Resistor_THT:R_Axial_DIN0207_L6.3mm_D2.5mm_P10.16mm_Horizontal; Manufacturer (none) -> Royal Ohm; Manufacturer Part No. (none) -> MF0W4FF1001A50; Supplier (none) -> Tayda; Supplier Part No. (none) -> A-2200
- R3: footprint (none) -> Resistor_THT:R_Axial_DIN0207_L6.3mm_D2.5mm_P10.16mm_Horizontal; Manufacturer (none) -> Royal Ohm; Manufacturer Part No. (none) -> MF0W4FF6800A50; Supplier (none) -> Tayda; Supplier Part No. (none) -> A-2281
- R6: footprint (none) -> Resistor_THT:R_Axial_DIN0207_L6.3mm_D2.5mm_P10.16mm_Horizontal; Manufacturer (none) -> Royal Ohm; Manufacturer Part No. (none) -> MF0W4FF4701A50; Supplier (none) -> Tayda; Supplier Part No. (none) -> A-2310
- R7: Manufacturer Part No. MF0W4FF1003A50 -> MF0W4FF1004A50; Supplier Part No. A-2248 -> A-2277
- R8: Manufacturer Part No. MF0W4FF1003A50 -> MF0W4FF4703A50; Supplier Part No. A-2248 -> A-2180
- R9: Manufacturer Part No. MF0W4FF1003A50 -> MF0W4FF1002A50; Supplier Part No. A-2248 -> A-2203
- U1: footprint (none) -> Package_DIP:DIP-14_W7.62mm_Socket; Manufacturer (none) -> VARIOUS; Manufacturer Part No. (none) -> TL074CN; Supplier (none) -> Tayda; Supplier Part No. (none) -> A-1138
Other:
- note removed: "TODO: Create BOM"

Commit message: Converted noise to use 2n3904
Parts:
- removed Q1: BC548, Package_TO_SOT_THT:TO-92_Inline, symbol Transistor_BJT:BC548
- added Q?: 2N3904, Package_TO_SOT_THT:TO-92_Inline, symbol Transistor_BJT:2N3904
- C3: value 1uF -> .1uF
- R1, R2: value 100k -> 1M
- R3: value 680 -> 1.5k
Connections:
- net GND: now also Q?.2 (B)
- net at C3.1, R1.2: now also Q?.1 (E)
Other:
- note added: "TODO: Update footprints and BOM"
Changed lines of the file:
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@@
     (rev "REV1")
     (company "Northridge Devices")
-    (comment 1 "Schematic by Moritz Klien")
+    (comment 1 "Based on Schematic by Moritz Klien")
   )
   (junction (at 77.47 77.47) (diameter 0) (color 0 0 0 0)
@@
   (wire (pts (xy 135.89 45.72) (xy 135.89 58.42))
     (stroke (width 0) (type default) (color 0 0 0 0))
+  )
+  (text "TODO: Update footprints and BOM" (at 66.04 66.04 0)
+    (effects (font (size 1.27 1.27)) (justify left bottom))
   )
   (symbol (lib_id "Device:R") (at 127 99.06 90) (mirror x) (unit 1)
@@
     (pin "TN")
   )
-  (symbol (lib_id "Transistor_BJT:BC548") (at 46.99 85.09 0) (mirror x) (unit 1)
-    (in_bom yes) (on_board yes) (fields_autoplaced)
-    (property "Reference" "Q1" (id 0) (at 52.07 83.8199 0)
-      (effects (font (size 1.27 1.27)) (justify left))
-    )
-    (property "Value" "BC548" (id 1) (at 52.07 86.3599 0)
+  (symbol (lib_id "Transistor_BJT:2N3904") (at 46.99 85.09 0) (mirror x) (unit 1)
+    (in_bom yes) (on_board yes) (fields_autoplaced)
+    (property "Reference" "Q?" (id 0) (at 52.07 83.8199 0)
+      (effects (font (size 1.27 1.27)) (justify left))
+    )
+    (property "Value" "2N3904" (id 1) (at 52.07 86.3599 0)
       (effects (font (size 1.27 1.27)) (justify left))
     )
@@
       (effects (font (size 1.27 1.27) italic) (justify left) hide)
     )
-    (property "Datasheet" "https://www.onsemi.com/pub/Collateral/BC550-D.pdf" (id 3) (at 46.99 85.09 0)
+    (property "Datasheet" "https://www.onsemi.com/pub/Collateral/2N3903-D.PDF" (id 3) (at 46.99 85.09 0)
       (effects (font (size 1.27 1.27)) (justify left) hide)
-    )
-    (property "Supplier" "Tayda" (id 4) (at 46.99 85.09 0)
-      (effects (font (size 1.27 1.27)) hide)
-    )
-    (property "Manufacturer" "KEC" (id 5) (at 46.99 85.09 0)
-      (effects (font (size 1.27 1.27)) hide)
-    )
-    (property "Manufacturer Part No." "BC548B" (id 6) (at 46.99 85.09 0)
-      (effects (font (size 1.27 1.27)) hide)
-    )
-    (property "Supplier Part No." "A-141" (id 7) (at 46.99 85.09 0)
-      (effects (font (size 1.27 1.27)) hide)
     )
     (pin "1")
@@
       (effects (font (size 1.27 1.27)) (justify right))
     )
-    (property "Value" "100k" (id 1) (at 52.07 72.3899 0)
+    (property "Value" "1M" (id 1) (at 52.07 72.3899 0)
       (effects (font (size 1.27 1.27)) (justify right))
     )
@@
     (in_bom yes) (on_board yes) (fields_autoplaced)
     (property "Reference" "C3" (id 0) (at 64.77 69.85 90))
-    (property "Value" "1uF" (id 1) (at 64.77 72.39 90))
+    (property "Value" ".1uF" (id 1) (at 64.77 72.39 90))
     (property "Footprint" "Capacitor_THT:C_Rect_L7.2mm_W3.5mm_P5.00mm_FKS2_FKP2_MKS2_MKP2" (id 2) (at 68.58 76.5048 0)
       (effects (font (size 1.27 1.27)) hide)
@@
       (effects (font (size 1.27 1.27)) (justify right))
     )
-    (property "Value" "100k" (id 1) (at 80.01 86.3599 0)
+    (property "Value" "1M" (id 1) (at 80.01 86.3599 0)
       (effects (font (size 1.27 1.27)) (justify right))
     )
@@
       (effects (font (size 1.27 1.27)) (justify left))
     )
-    (property "Value" "680" (id 1) (at 93.98 99.0599 0)
+    (property "Value" "1.5k" (id 1) (at 93.98 99.0599 0)
       (effects (font (size 1.27 1.27)) (justify left))
     )
@@
     )
     (path "/7ba5dc36-6c50-47a6-b441-5dddf850725d"
-      (reference "C3") (unit 1) (value "1uF") (footprint "Capacitor_THT:C_Rect_L7.2mm_W3.5mm_P5.00mm_FKS2_FKP2_MKS2_MKP2")
+      (reference "C3") (unit 1) (value ".1uF") (footprint "Capacitor_THT:C_Rect_L7.2mm_W3.5mm_P5.00mm_FKS2_FKP2_MKS2_MKP2")
     )
     (path "/2699e0e0-da3e-4405-b53d-6667e01615e0"
@@
       (reference "J4") (unit 1) (value "PINK_OUT") (footprint "Tayda_Jacks:PJ-323M")
     )
-    (path "/3d01dbdc-9bc3-4ee1-a4bf-6d3be55846a4"
-      (reference "Q1") (unit 1) (value "BC548") (footprint "Package_TO_SOT_THT:TO-92_Inline")
+    (path "/354628aa-0d46-43f4-8897-2147f15a3720"
+      (reference "Q?") (unit 1) (value "2N3904") (footprint "Package_TO_SOT_THT:TO-92_Inline")
     )
     (path "/4df10721-607d-49ab-b396-d5ca6de9163e"
-      (reference "R1") (unit 1) (value "100k") (footprint "Resistor_THT:R_Axial_DIN0207_L6.3mm_D2.5mm_P10.16mm_Horizontal")
+      (reference "R1") (unit 1) (value "1M") (footprint "Resistor_THT:R_Axial_DIN0207_L6.3mm_D2.5mm_P10.16mm_Horizontal")
     )
     (path "/b6d1ed76-de4f-4c4d-b209-032b989640fc"
-      (reference "R2") (unit 1) (value "100k") (footprint "Resistor_THT:R_Axial_DIN0207_L6.3mm_D2.5mm_P10.16mm_Horizontal")
+      (reference "R2") (unit 1) (value "1M") (footprint "Resistor_THT:R_Axial_DIN0207_L6.3mm_D2.5mm_P10.16mm_Horizontal")
     )
     (path "/bddfd24d-d893-473c-99e9-1ff42708b1de"
-      (reference "R3") (unit 1) (value "680") (footprint "Resistor_THT:R_Axial_DIN0207_L6.3mm_D2.5mm_P10.16mm_Horizontal")
+      (reference "R3") (unit 1) (value "1.5k") (footprint "Resistor_THT:R_Axial_DIN0207_L6.3mm_D2.5mm_P10.16mm_Horizontal")
     )
     (path "/08d291a6-f9ac-429a-8f92-c7f657c7ea3c"
